Commit message: Create my robot.

File: sugar_description/urdf/sugar_robot.xacro (robot description, xacro)
@@ -3,5 +3,5 @@
   <xacro:property name="PI" value="3.1415926535897931"/>
   <!-- import gazebo reference -->
-  <xacro:include filename="$(find sugar_description)/xacro/sugar_robot.gazebo"/>
+  <xacro:include filename="$(find sugar_description)/urdf/sugar_robot.gazebo"/>
   <!-- import livox 3D-lidar model -->
   <xacro:include filename="$(find ros2_livox_simulation)/urdf/mid360.xacro"/>
@@ -33,4 +33,9 @@
       </geometry>
     </collision>
+    <inertial>
+      <mass value="27.1"/>
+      <origin xyz="-0.1995 0.0 0.19" rpy="0.0 0.0 0.0"/>
+      <inertia ixx="0.78032248125" ixy="0.0" ixz="0.0" iyy="0.883913925" iyz="0.0" izz="1.25773640625"/>
+    </inertial>
   </link>
   <!-- 3D-lidar stand -->
@@ -81,9 +86,10 @@
   </link>-->
   <!-- left wheel -->
-  <joint name="left_wheel_joint" type="continuous">
+  <joint name="left_wheel_hinge" type="revolute">
     <parent link="base_link"/>
     <child link="left_wheel"/>
-    <origin xyz="0.0 0.3 0.0" rpy="1.57079632679 0 0"/>
+    <origin xyz="0.0 0.3 0.0" rpy="0.0 1.57079632679 1.57079632679"/>
     <axis xyz="0 0 1"/>
+    <limit effort="100" velocity="100.0" lower="-5000" upper="5000"/>
   </joint>
   <link name="left_wheel">
@@ -91,23 +97,29 @@
       <origin xyz="0.0 0.0 0.0" rpy="0 0 0"/>
       <geometry>
-        <cylinder radius="0.1" length="0.08"/>
-      </geometry>
-      <material name="white">
-        <color rgba="1.0 1.0 1.0 1.0"/>
-      </material>
-    </visual>
-    <collision>
-      <origin xyz="0.0 0.0 0.0" rpy="0 0 0"/>
-      <geometry>
-        <cylinder radius="0.1" length="0.05"/>
-      </geometry>
-    </collision>
+        <cylinder radius="0.1015" length="0.047"/>
+      </geometry>
+      <material name="white">
+        <color rgba="1.0 1.0 1.0 1.0"/>
+      </material>
+    </visual>
+    <collision>
+      <origin xyz="0.0 0.0 0.0" rpy="0 0 0"/>
+      <geometry>
+        <cylinder radius="0.1015" length="0.047"/>
+      </geometry>
+    </collision>
+    <inertial>
+      <mass value="3.4"/>
+      <origin xyz="0.0 0.0 0.0" rpy="0.0 1.57079632679 1.57079632679"/>
+      <inertia ixx="0.00938279583" ixy="0.0" ixz="0.0" iyy="0.00938279583" iyz="0.0" izz="0.017513825"/>
+    </inertial>
   </link>
   <!-- right wheel -->
-  <joint name="right_wheel_joint" type="continuous">
+  <joint name="right_wheel_hinge" type="revolute">
     <parent link="base_link"/>
     <child link="right_wheel"/>
-    <origin xyz="0.0 -0.3 0.0" rpy="1.57079632679 0 0"/>
+    <origin xyz="0.0 -0.3 0.0" rpy="0.0 1.57079632679 1.57079632679"/>
     <axis xyz="0 0 1"/>
+    <limit effort="100" velocity="100.0" lower="-5000" upper="5000"/>
   </joint>
   <link name="right_wheel">
@@ -115,24 +127,29 @@
       <origin xyz="0.0 0.0 0.0" rpy="0 0 0"/>
       <geometry>
-        <cylinder radius="0.1" length="0.08"/>
-      </geometry>
-      <material name="white">
-        <color rgba="1.0 1.0 1.0 1.0"/>
-      </material>
-    </visual>
-    <collision>
-      <origin xyz="0.0 0.0 0.0" rpy="0 0 0"/>
-      <geometry>
-        <cylinder radius="0.1" length="0.05"/>
-      </geometry>
-    </collision>
+        <cylinder radius="0.1015" length="0.047"/>
+      </geometry>
+      <material name="white">
+        <color rgba="1.0 1.0 1.0 1.0"/>
+      </material>
+    </visual>
+    <collision>
+      <origin xyz="0.0 0.0 0.0" rpy="0 0 0"/>
+      <geometry>
+        <cylinder radius="0.1015" length="0.047"/>
+      </geometry>
+    </collision>
+    <inertial>
+      <mass value="3.4"/>
+      <origin xyz="0.0 0.0 0.0" rpy="0.0 1.57079632679 1.57079632679"/>
+      <inertia ixx="0.00938279583" ixy="0.0" ixz="0.0" iyy="0.00938279583" iyz="0.0" izz="0.017513825"/>
+    </inertial>
   </link>
   <!-- front left caster -->
   <joint name="front_left_caster_hinge" type="fixed">
     <parent link="base_link"/>
-    <child link="front_left_caster_link"/>
+    <child link="front_left_caster"/>
     <origin xyz="0.2 0.15 -0.05" rpy="0.0 0.0 0.0"/>
   </joint>
-  <link name="front_left_caster_link">
+  <link name="front_left_caster">
     <visual>
       <origin xyz="0.0 0.0 0.0" rpy="0.0 0.0 0.0"/>
@@ -154,8 +171,8 @@
   <joint name="front_right_caster_hinge" type="fixed">
     <parent link="base_link"/>
-    <child link="front_right_caster_link"/>
+    <child link="front_right_caster"/>
     <origin xyz="0.2 -0.15 -0.05" rpy="0.0 0.0 0.0"/>
   </joint>
-  <link name="front_right_caster_link">
+  <link name="front_right_caster">
     <visual>
       <origin xyz="0.0 0.0 0.0" rpy="0.0 0.0 0.0"/>
@@ -177,8 +194,8 @@
   <joint name="rear_left_caster_hinge" type="fixed">
     <parent link="base_link"/>
-    <child link="rear_left_caster_link"/>
+    <child link="rear_left_caster"/>
     <origin xyz="-0.35 0.15 -0.05" rpy="0.0 0.0 0.0"/>
   </joint>
-  <link name="rear_left_caster_link">
+  <link name="rear_left_caster">
     <visual>
       <origin xyz="0.0 0.0 0.0" rpy="0.0 0.0 0.0"/>
@@ -200,8 +217,8 @@
   <joint name="rear_right_caster_hinge" type="fixed">
     <parent link="base_link"/>
-    <child link="rear_right_caster_link"/>
+    <child link="rear_right_caster"/>
     <origin xyz="-0.35 -0.15 -0.05" rpy="0.0 0.0 0.0"/>
   </joint>
-  <link name="rear_right_caster_link">
+  <link name="rear_right_caster">
     <visual>
       <origin xyz="0.0 0.0 0.0" rpy="0.0 0.0 0.0"/>

Commit message: Restore urdf file of my robot.

File: sugar_description/urdf/sugar_robot.xacro (robot description, xacro)
@@ -5,8 +5,12 @@
   <xacro:include filename="$(find sugar_description)/urdf/sugar_robot.gazebo"/>
   <!-- import livox 3D-lidar model -->
-  <xacro:include filename="$(find ros2_livox_simulation)/urdf/mid360.xacro"/>
+  <xacro:include filename="$(find sugar_description)/urdf/livox.xacro"/>
+  <xacro:sensor_livox name="livox" parent="lidar_stand" min_angle="-2.35619" max_angle="2.35619" samples="720">
+    <origin xyz="0.1 0.0 0.35" rpy="3.1415926535897931 0 0"/>
+  </xacro:sensor_livox>
+  <!--<xacro:include filename="$(find ros2_livox_simulation)/urdf/mid360.xacro"/>
   <xacro:mid360 name="livox" parent="lidar_stand" topic="mid360">
     <origin xyz="0.1 0 0.35" rpy="0 0 0"/>
-  </xacro:mid360>
+  </xacro:mid360>-->
   <!-- base footprint -->
   <link name="base_footprint"/>
